File: PCB/Oscilloscope.kicad_pcb (KiCad board)
At the start: 2 copper layers, 99.6 x 57.8 mm, 17 parts, among them J1 Left Header, J2 Right Header, J3 Conn_01x08, J4 Conn_01x02, SW1 RotaryEncoder_Switch, SW2 RotaryEncoder_Switch, U1 MCP6002-xP

Commit message: Add files via upload
Routing:
- net GND: track 184.6 -> 0.00 mm
- added copper zone on B.Cu, net GND
- added copper zone on F.Cu, net GND
Changed lines of the file:
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@@
-	)
-	(segment
-		(start 122.7278 76.678635)
-		(end 128.322365 82.2732)
-		(width 0.2)
-		(layer "F.Cu")
-		(net "GND")
-	)
-	(segment
-		(start 98.9584 68.5584)
-		(end 98.9584 58.674)
-		(width 0.2)
-		(layer "F.Cu")
-		(net "GND")
-	)
-	(segment
-		(start 133.778 77.1232)
-		(end 133.778 81.1732)
-		(width 0.2)
-		(layer "F.Cu")
-		(net "GND")
-	)
-	(segment
-		(start 72.136 72.3684)
-		(end 69.636 74.8684)
-		(width 0.2)
-		(layer "F.Cu")
-		(net "GND")
-	)
-	(segment
-		(start 122.7278 76.6265)
-		(end 118.5421 72.4408)
-		(width 0.2)
-		(layer "F.Cu")
-		(net "GND")
-	)
-	(segment
-		(start 132.678 82.2732)
-		(end 133.778 81.1732)
-		(width 0.2)
-		(layer "F.Cu")
-		(net "GND")
-	)
-	(segment
-		(start 109.0676 48.5648)
-		(end 109.1692 48.5648)
-		(width 0.2)
-		(layer "F.Cu")
-		(net "GND")
-	)
-	(segment
-		(start 133.778 64.9732)
-		(end 133.778 69.0232)
-		(width 0.2)
-		(layer "F.Cu")
-		(net "GND")
-	)
-	(segment
-		(start 133.778 69.0232)
-		(end 133.778 73.0732)
-		(width 0.2)
-		(layer "F.Cu")
-		(net "GND")
-	)
-	(segment
-		(start 148.3868 55.4228)
-		(end 148.3868 30.0228)
-		(width 0.2)
-		(layer "F.Cu")
-		(net "GND")
-	)
-	(segment
-		(start 95.1484 72.3684)
-		(end 98.9584 68.5584)
-		(width 0.2)
-		(layer "F.Cu")
-		(net "GND")
-	)
-	(segment
-		(start 128.322365 82.2732)
-		(end 132.678 82.2732)
-		(width 0.2)
-		(layer "F.Cu")
-		(net "GND")
-	)
-	(segment
-		(start 98.9584 58.674)
-		(end 109.0676 48.5648)
-		(width 0.2)
-		(layer "F.Cu")
-		(net "GND")
-	)
-	(segment
-		(start 122.7278 67.3658)
-		(end 123.9012 66.1924)
-		(width 0.2)
-		(layer "F.Cu")
-		(net "GND")
-	)
-	(segment
-		(start 74.636 74.8684)
-		(end 80.6484 74.8684)
-		(width 0.2)
-		(layer "F.Cu")
-		(net "GND")
-	)
-	(segment
-		(start 100.1776 72.4408)
-		(end 95.2208 72.4408)
-		(width 0.2)
-		(layer "F.Cu")
-		(net "GND")
-	)
-	(segment
-		(start 122.7278 76.6265)
-		(end 122.7278 67.3658)
-		(width 0.2)
-		(layer "F.Cu")
-		(net "GND")
-	)
-	(segment
-		(start 133.778 73.0732)
-		(end 133.778 77.1232)
-		(width 0.2)
-		(layer "F.Cu")
-		(net "GND")
-	)
-	(segment
-		(start 69.636 74.8684)
-		(end 57.636 74.8684)
-		(width 0.2)
-		(layer "F.Cu")
-		(net "GND")
-	)
-	(segment
-		(start 95.2208 72.4408)
-		(end 95.1484 72.3684)
-		(width 0.2)
-		(layer "F.Cu")
-		(net "GND")
-	)
-	(segment
-		(start 118.5421 72.4408)
-		(end 107.7976 72.4408)
-		(width 0.2)
-		(layer "F.Cu")
-		(net "GND")
-	)
-	(segment
-		(start 95.1484 72.3684)
-		(end 92.6484 74.8684)
-		(width 0.2)
-		(layer "F.Cu")
-		(net "GND")
-	)
-	(segment
-		(start 122.7278 76.6265)
-		(end 122.7278 76.678635)
-		(width 0.2)
-		(layer "F.Cu")
-		(net "GND")
-	)
-	(segment
-		(start 92.6484 74.8684)
-		(end 80.6484 74.8684)
-		(width 0.2)
-		(layer "F.Cu")
-		(net "GND")
-	)
-	(segment
-		(start 72.136 72.3684)
-		(end 74.636 74.8684)
-		(width 0.2)
-		(layer "F.Cu")
-		(net "GND")
-	)
-	(segment
-		(start 138.8364 64.9732)
-		(end 133.778 64.9732)
-		(width 0.2)
-		(layer "B.Cu")
-		(net "GND")
-	)
-	(segment
-		(start 100.1776 72.4408)
-		(end 107.7976 72.4408)
-		(width 0.2)
-		(layer "B.Cu")
-		(net "GND")
-	)
-	(segment
-		(start 148.3868 55.4228)
-		(end 138.8364 64.9732)
-		(width 0.2)
-		(layer "B.Cu")
-		(net "GND")
 	)
 	(segment
@@
 		(net "/BLK")
 	)
+	(zone
+		(net "GND")
+		(layers "F.Cu" "B.Cu")
+		(name "GND")
+		(hatch edge 0.5)
+		(connect_pads
+			(clearance 0.5)
+		)
+		(min_thickness 0.25)
+		(fill yes
+			(thermal_gap 0.5)
+			(thermal_bridge_width 0.5)
+			(island_removal_mode 0)
+		)
+		(polygon
+			(pts
+				(xy 70.612 28.3972) (xy 55.8292 28.4988) (xy 55.5752 83.4136) (xy 110.8964 84.6328) (xy 153.416 84.2772)
+				(xy 153.5684 28.3464) (xy 152.0444 27.8892)
+			)
+		)
+	)
 	(embedded_fonts no)

Commit message: Add files via upload
Parts:
- removed the REF** at (103.0, 48.8)
Changed lines of the file:
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@@
-	(footprint "MountingHole:MountingHole_3.2mm_M3"
-		(layer "F.Cu")
-		(at 102.9716 48.8188)
-		(descr "Mounting Hole 3.2mm, M3, no annular, generated by kicad-footprint-generator mountinghole.py")
-		(tags "mountinghole M3")
-		(property "Reference" "REF**"
-			(at 0 -4.15 0)
-			(layer "F.SilkS")
-			(effects
-				(font
-					(size 1 1)
-					(thickness 0.15)
-				)
-			)
-		)
-		(property "Value" "MountingHole_3.2mm_M3"
-			(at 0 4.15 0)
-			(layer "F.Fab")
-			(effects
-				(font
-					(size 1 1)
-					(thickness 0.15)
-				)
-			)
-		)
-		(property "Datasheet" ""
-			(at 0 0 0)
-			(layer "F.Fab")
-			(hide yes)
-			(effects
-				(font
-					(size 1.27 1.27)
-				)
-			)
-		)
-		(property "Description" ""
-			(at 0 0 0)
-			(layer "F.Fab")
-			(hide yes)
-			(effects
-				(font
-					(size 1.27 1.27)
-				)
-			)
-		)
-		(property "KiLib_Generator" "mounting_hardware/mounting_hole"
-			(at 0 0 0)
-			(layer "F.SilkS")
-			(hide yes)
-			(effects
-				(font
-					(size 1 1)
-					(thickness 0.15)
-				)
-			)
-		)
-		(attr exclude_from_pos_files exclude_from_bom)
-		(duplicate_pad_numbers_are_jumpers no)
-		(fp_circle
-			(center 0 0)
-			(end 3.2 0)
-			(stroke
-				(width 0.15)
-				(type solid)
-			)
-			(fill no)
-			(layer "Cmts.User")
-		)
-		(fp_circle
-			(center 0 0)
-			(end 3.45 0)
-			(stroke
-				(width 0.05)
-				(type solid)
-			)
-			(fill no)
-			(layer "F.CrtYd")
-		)
-		(fp_text user "${REFERENCE}"
-			(at 0 0 0)
-			(layer "F.Fab")
-			(effects
-				(font
-					(size 1 1)
-					(thickness 0.15)
-				)
-			)
-		)
-		(pad "" np_thru_hole circle
-			(at 0 0)
-			(size 3.2 3.2)
-			(drill 3.2)
-			(layers "*.Cu" "*.Mask")
-		)
-		(embedded_fonts no)
-	)
 	(footprint "MountingHole:MountingHole_3.2mm_M3"
 		(layer "F.Cu")
